File: Bottom/ZIF socket grande/bootloader_burner.sch (EAGLE design)
At the start: 7 parts, among them Y1 16MHz

Commit message: Cambie el diseño de la plaqueta con zif socket grande para que queden ordenados los pines con los del Arduino. Tambien cambie el dieño de la plaqueta doble (que igual hay que cambiarla poque la gracia de esa es que quede montada en el Arduino)
Connections:
- net N$1 renamed PIN_13_ARDUINO
- net N$2 renamed PIN_12_ARDUINO
- net N$3 renamed PIN_11_ARDUINO
- net N$6 renamed PIN_10_ARDUINO
Changed lines of the file:
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@@
 </segment>
 </net>
-<net name="N$6" class="0">
+<net name="PIN_10_ARDUINO" class="0">
 <segment>
 <wire x1="38.1" y1="76.2" x2="38.1" y2="83.82" width="0.1524" layer="91"/>
@@
 </segment>
 </net>
-<net name="N$1" class="0">
+<net name="PIN_13_ARDUINO" class="0">
 <segment>
 <pinref part="ZX1" gate="G$1" pin="19"/>
@@
 </segment>
 </net>
-<net name="N$2" class="0">
+<net name="PIN_12_ARDUINO" class="0">
 <segment>
 <pinref part="ZX1" gate="G$1" pin="18"/>
@@
 </segment>
 </net>
-<net name="N$3" class="0">
+<net name="PIN_11_ARDUINO" class="0">
 <segment>
 <pinref part="ZX1" gate="G$1" pin="17"/>
