File: Bottom/ZIF socket grande/bootloader_burner.brd (EAGLE design)
At the start: 57 x 53.3 mm, 7 parts, among them Y1 16MHz

Commit message: Cambie el diseño de la plaqueta con zif socket grande para que queden ordenados los pines con los del Arduino. Tambien cambie el dieño de la plaqueta doble (que igual hay que cambiarla poque la gracia de esa es que quede montada en el Arduino)
Parts:
- moved JP2 9.18 mm to (39.4, 37.6), turned to 180 degrees
- moved JP1 1.44 mm to (26.9, 46.0), turned to 180 degrees
Connections:
- net N$1 renamed PIN_13_ARDUINO
- net N$2 renamed PIN_12_ARDUINO
- net N$3 renamed PIN_11_ARDUINO
- net N$6 renamed PIN_10_ARDUINO
Routing:
- net PIN_13_ARDUINO: track 31.3 -> 14.3 mm
- net PIN_10_ARDUINO: track 51.8 -> 44.7 mm
- net PIN_11_ARDUINO: track 31.3 -> 37.6 mm
- net GND: track 132.9 -> 138.0 mm
- net PIN_12_ARDUINO: track 31.3 -> 27.8 mm
- net VCC: track 133.4 -> 134.3 mm
Other:
- board text added: "13-12-11-10"
- board text removed: "10 / 11 / 12 / 13"
Changed lines of the file:
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@@
 <wire x1="66.04" y1="51.816" x2="64.516" y2="53.34" width="0" layer="20"/>
 <wire x1="64.516" y1="53.34" x2="11.557" y2="53.34" width="0" layer="20"/>
-<text x="25.146" y="49.53" size="1.778" layer="16" rot="MR0">VCC</text>
-<text x="36.068" y="49.53" size="1.778" layer="16" rot="MR0">GND</text>
-<text x="52.832" y="43.18" size="1.778" layer="16" rot="MR0">10 / 11 / 12 / 13</text>
 <hole x="15.24" y="49.53" drill="0.1778"/>
 <hole x="63.246" y="50.038" drill="0.1778"/>
@@
 <hole x="66.04" y="2.54" drill="0.1778"/>
 <hole x="24.892" y="32.258" drill="0.1778"/>
-<hole x="49.53" y="39.37" drill="0.1778"/>
+<text x="42.926" y="31.75" size="1.778" layer="16" rot="MR0">13-12-11-10</text>
+<text x="22.86" y="44.704" size="1.778" layer="16" rot="MR0">GND</text>
+<text x="36.576" y="44.704" size="1.778" layer="16" rot="MR0">VCC</text>
 </plain>
 <attributes>
@@
 <attribute name="VALUE" x="57.404" y="32.766" size="0.6096" layer="27" font="vector" ratio="20" align="top-center"/>
 </element>
-<element name="JP2" library="pinhead" library_urn="urn:adsk.eagle:library:325" package="1X04" package3d_urn="urn:adsk.eagle:package:22407/2" value="" x="30.48" y="39.878" smashed="yes">
-<attribute name="NAME" x="25.3238" y="41.7068" size="1.27" layer="25" ratio="10"/>
-<attribute name="POPULARITY" value="91" x="30.48" y="39.878" size="1.778" layer="27" display="off"/>
-<attribute name="VALUE" x="25.4" y="36.703" size="1.27" layer="27"/>
-</element>
-<element name="JP1" library="pinhead" library_urn="urn:adsk.eagle:library:325" package="1X02" package3d_urn="urn:adsk.eagle:package:22435/2" value="" x="27.94" y="46.99" smashed="yes">
-<attribute name="NAME" x="25.3238" y="48.8188" size="1.27" layer="25" ratio="10"/>
-<attribute name="POPULARITY" value="98" x="27.94" y="46.99" size="1.778" layer="27" display="off"/>
-<attribute name="VALUE" x="25.4" y="43.815" size="1.27" layer="27"/>
+<element name="JP2" library="pinhead" library_urn="urn:adsk.eagle:library:325" package="1X04" package3d_urn="urn:adsk.eagle:package:22407/2" value="" x="39.37" y="37.592" smashed="yes" rot="R180">
+<attribute name="NAME" x="44.5262" y="35.7632" size="1.27" layer="25" ratio="10" rot="R180"/>
+<attribute name="POPULARITY" value="91" x="39.37" y="37.592" size="1.778" layer="27" rot="R180" display="off"/>
+<attribute name="VALUE" x="44.45" y="40.767" size="1.27" layer="27" rot="R180"/>
+</element>
+<element name="JP1" library="pinhead" library_urn="urn:adsk.eagle:library:325" package="1X02" package3d_urn="urn:adsk.eagle:package:22435/2" value="" x="26.924" y="45.974" smashed="yes" rot="R180">
+<attribute name="NAME" x="29.5402" y="44.1452" size="1.27" layer="25" ratio="10" rot="R180"/>
+<attribute name="POPULARITY" value="98" x="26.924" y="45.974" size="1.778" layer="27" rot="R180" display="off"/>
+<attribute name="VALUE" x="29.464" y="49.149" size="1.27" layer="27" rot="R180"/>
 </element>
 <element name="ZX1" library="con-3m" library_urn="urn:adsk.eagle:library:119" package="228-1277-00-0602J" package3d_urn="urn:adsk.eagle:package:5569/1" value="228-1277-00-0602J" x="40.132" y="17.018" smashed="yes">
@@
 <wire x1="17.78" y1="41.656" x2="14.986" y2="38.862" width="1.524" layer="16"/>
 <contactref element="JP1" pad="1"/>
-<wire x1="26.67" y1="46.99" x2="19.304" y2="46.99" width="1.524" layer="16"/>
-<wire x1="19.304" y1="46.99" x2="17.78" y2="45.466" width="1.524" layer="16"/>
-<wire x1="17.78" y1="45.466" x2="17.78" y2="41.656" width="1.524" layer="16"/>
 <contactref element="ZX1" pad="20"/>
 <contactref element="ZX1" pad="7"/>
@@
 <wire x1="22.098" y1="28.956" x2="20.828" y2="27.686" width="1.524" layer="16"/>
 <wire x1="23.114" y1="17.018" x2="35.306" y2="17.018" width="1.524" layer="16"/>
+<wire x1="17.78" y1="41.656" x2="27.432" y2="41.656" width="1.524" layer="16"/>
+<wire x1="27.432" y1="41.656" x2="28.194" y2="42.418" width="1.524" layer="16"/>
+<wire x1="28.194" y1="42.418" x2="28.194" y2="45.974" width="1.524" layer="16"/>
 </signal>
 <signal name="GND">
@@
 <wire x1="59.944" y1="47.244" x2="59.944" y2="48.514" width="1.524" layer="16"/>
 <wire x1="59.944" y1="48.514" x2="59.182" y2="49.276" width="1.524" layer="16"/>
-<wire x1="38.608" y1="49.276" x2="36.068" y2="46.736" width="1.524" layer="16"/>
-<wire x1="36.068" y1="46.736" x2="29.464" y2="46.736" width="1.524" layer="16"/>
-<wire x1="29.464" y1="46.736" x2="29.21" y2="46.99" width="1.524" layer="16"/>
-<wire x1="59.182" y1="49.276" x2="38.608" y2="49.276" width="1.524" layer="16"/>
 <wire x1="63.246" y1="43.942" x2="59.944" y2="47.244" width="1.524" layer="16"/>
 <wire x1="63.246" y1="36.83" x2="63.246" y2="43.942" width="1.524" layer="16"/>
+<wire x1="26.67" y1="49.276" x2="25.654" y2="48.26" width="1.524" layer="16"/>
+<wire x1="25.654" y1="48.26" x2="25.654" y2="45.974" width="1.524" layer="16"/>
+<wire x1="59.182" y1="49.276" x2="26.67" y2="49.276" width="1.524" layer="16"/>
 <wire x1="59.944" y1="44.704" x2="55.245" y2="44.704" width="0" layer="19" extent="1-1"/>
 </signal>
@@
 <wire x1="48.26" y1="15.24" x2="46.482" y2="13.462" width="1.524" layer="16"/>
 </signal>
-<signal name="N$6">
+<signal name="PIN_10_ARDUINO">
 <contactref element="R1" pad="2"/>
-<wire x1="17.78" y1="31.496" x2="22.352" y2="36.068" width="1.524" layer="16"/>
-<wire x1="22.352" y1="36.068" x2="22.352" y2="41.402" width="1.524" layer="16"/>
-<wire x1="22.352" y1="41.402" x2="24.384" y2="43.434" width="1.524" layer="16"/>
 <contactref element="JP2" pad="4"/>
-<wire x1="34.29" y1="39.878" x2="34.29" y2="41.656" width="1.524" layer="16"/>
-<wire x1="32.512" y1="43.434" x2="24.384" y2="43.434" width="1.524" layer="16"/>
-<wire x1="34.29" y1="41.656" x2="32.512" y2="43.434" width="1.524" layer="16"/>
 <contactref element="ZX1" pad="1"/>
 <wire x1="23.368" y1="9.398" x2="23.622" y2="9.398" width="1.524" layer="16"/>
 <wire x1="23.368" y1="9.398" x2="18.288" y2="14.478" width="1.524" layer="16"/>
-<wire x1="18.288" y1="30.988" x2="17.78" y2="31.496" width="1.524" layer="16"/>
 <wire x1="18.288" y1="14.478" x2="18.288" y2="30.988" width="1.524" layer="16"/>
-</signal>
-<signal name="N$1">
+<wire x1="17.78" y1="31.496" x2="18.288" y2="30.988" width="1.524" layer="16"/>
+<wire x1="18.288" y1="30.988" x2="24.892" y2="37.592" width="1.524" layer="16"/>
+<wire x1="24.892" y1="37.592" x2="35.56" y2="37.592" width="1.524" layer="16"/>
+</signal>
+<signal name="PIN_13_ARDUINO">
 <contactref element="ZX1" pad="19"/>
 <contactref element="JP2" pad="1"/>
-<wire x1="46.482" y1="24.638" x2="46.482" y2="29.718" width="1.524" layer="16"/>
-<wire x1="46.482" y1="29.718" x2="44.704" y2="31.496" width="1.524" layer="16"/>
-<wire x1="31.242" y1="31.496" x2="26.67" y2="36.068" width="1.524" layer="16"/>
-<wire x1="26.67" y1="36.068" x2="26.67" y2="39.878" width="1.524" layer="16"/>
-<wire x1="44.704" y1="31.496" x2="31.242" y2="31.496" width="1.524" layer="16"/>
-</signal>
-<signal name="N$2">
+<wire x1="46.482" y1="34.29" x2="43.18" y2="37.592" width="1.524" layer="16"/>
+<wire x1="46.482" y1="24.638" x2="46.482" y2="34.29" width="1.524" layer="16"/>
+</signal>
+<signal name="PIN_12_ARDUINO">
 <contactref element="ZX1" pad="18"/>
 <contactref element="JP2" pad="2"/>
-<wire x1="49.022" y1="24.638" x2="49.022" y2="30.734" width="1.524" layer="16"/>
-<wire x1="32.258" y1="34.036" x2="29.21" y2="37.084" width="1.524" layer="16"/>
-<wire x1="29.21" y1="37.084" x2="29.21" y2="39.878" width="1.524" layer="16"/>
-<wire x1="49.022" y1="30.734" x2="45.72" y2="34.036" width="1.524" layer="16"/>
-<wire x1="45.72" y1="34.036" x2="32.258" y2="34.036" width="1.524" layer="16"/>
-</signal>
-<signal name="N$3">
+<wire x1="49.022" y1="24.638" x2="49.022" y2="40.132" width="1.524" layer="16"/>
+<wire x1="41.91" y1="41.656" x2="40.64" y2="40.386" width="1.524" layer="16"/>
+<wire x1="40.64" y1="40.386" x2="40.64" y2="37.592" width="1.524" layer="16"/>
+<wire x1="49.022" y1="40.132" x2="47.498" y2="41.656" width="1.524" layer="16"/>
+<wire x1="47.498" y1="41.656" x2="41.91" y2="41.656" width="1.524" layer="16"/>
+</signal>
+<signal name="PIN_11_ARDUINO">
 <contactref element="ZX1" pad="17"/>
 <contactref element="JP2" pad="3"/>
-<wire x1="51.562" y1="24.638" x2="51.562" y2="31.75" width="1.524" layer="16"/>
-<wire x1="33.274" y1="36.576" x2="31.75" y2="38.1" width="1.524" layer="16"/>
-<wire x1="31.75" y1="38.1" x2="31.75" y2="39.878" width="1.524" layer="16"/>
-<wire x1="51.562" y1="31.75" x2="46.736" y2="36.576" width="1.524" layer="16"/>
-<wire x1="46.736" y1="36.576" x2="33.274" y2="36.576" width="1.524" layer="16"/>
+<wire x1="51.562" y1="42.164" x2="49.276" y2="44.45" width="1.524" layer="16"/>
+<wire x1="51.562" y1="24.638" x2="51.562" y2="42.164" width="1.524" layer="16"/>
+<wire x1="49.276" y1="44.45" x2="40.132" y2="44.45" width="1.524" layer="16"/>
+<wire x1="40.132" y1="44.45" x2="38.1" y2="42.418" width="1.524" layer="16"/>
+<wire x1="38.1" y1="42.418" x2="38.1" y2="37.592" width="1.524" layer="16"/>
 </signal>
 </signals>

Commit message: Agregue las dos plaquetas simples al word. Pase el word a pdf y lo uni con los planos a imprimir de los circuitos
Routing:
- net GND: track 138.0 -> 142.7 mm
- net VCC: track 134.3 -> 137.9 mm
Other:
- board size 57 x 53.3 mm -> 58.5 x 53.3 mm
