File: Bottom/ZIF socket chico/bootloader_burner.sch (EAGLE design)
At the start: 6 parts, among them J1 ZIFSOCKET-28-3", Y1 16MHz

Commit message: Cambie la plaqueta para el zif socket chico para que queden ordenados los pines para conectar la plaqueta al Arduino
Connections:
- net PIN10ARDUINO: now also JP3.10; no longer JP3.1
- net PIN11ARDUINO: now also JP3.7; no longer JP3.10
- net PIN12ARDUINO: now also JP3.4; no longer JP3.7
- net PIN13ARDUINO: now also JP3.1; no longer JP3.4
Changed lines of the file:
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@@
 <pinref part="J1" gate="G$1" pin="P$17"/>
 <wire x1="91.44" y1="20.32" x2="71.12" y2="20.32" width="0.1524" layer="91"/>
-<wire x1="91.44" y1="20.32" x2="91.44" y2="63.5" width="0.1524" layer="91"/>
-<pinref part="JP3" gate="A" pin="10"/>
-<wire x1="91.44" y1="63.5" x2="116.84" y2="63.5" width="0.1524" layer="91"/>
+<wire x1="91.44" y1="20.32" x2="91.44" y2="71.12" width="0.1524" layer="91"/>
+<pinref part="JP3" gate="A" pin="7"/>
+<wire x1="91.44" y1="71.12" x2="116.84" y2="71.12" width="0.1524" layer="91"/>
 </segment>
 </net>
@@
 <pinref part="J1" gate="G$1" pin="P$18"/>
 <wire x1="88.9" y1="25.4" x2="71.12" y2="25.4" width="0.1524" layer="91"/>
-<wire x1="88.9" y1="25.4" x2="88.9" y2="71.12" width="0.1524" layer="91"/>
-<pinref part="JP3" gate="A" pin="7"/>
-<wire x1="88.9" y1="71.12" x2="116.84" y2="71.12" width="0.1524" layer="91"/>
+<wire x1="88.9" y1="25.4" x2="88.9" y2="78.74" width="0.1524" layer="91"/>
+<pinref part="JP3" gate="A" pin="4"/>
+<wire x1="88.9" y1="78.74" x2="116.84" y2="78.74" width="0.1524" layer="91"/>
 </segment>
 </net>
@@
 <pinref part="J1" gate="G$1" pin="P$19"/>
 <wire x1="86.36" y1="30.48" x2="71.12" y2="30.48" width="0.1524" layer="91"/>
-<wire x1="86.36" y1="30.48" x2="86.36" y2="78.74" width="0.1524" layer="91"/>
-<pinref part="JP3" gate="A" pin="4"/>
-<wire x1="86.36" y1="78.74" x2="116.84" y2="78.74" width="0.1524" layer="91"/>
+<wire x1="86.36" y1="30.48" x2="86.36" y2="86.36" width="0.1524" layer="91"/>
+<pinref part="JP3" gate="A" pin="1"/>
+<wire x1="86.36" y1="86.36" x2="116.84" y2="86.36" width="0.1524" layer="91"/>
 </segment>
 </net>
@@
 <segment>
 <pinref part="J1" gate="G$1" pin="P$1"/>
-<wire x1="38.1" y1="76.2" x2="38.1" y2="86.36" width="0.1524" layer="91"/>
-<wire x1="38.1" y1="86.36" x2="116.84" y2="86.36" width="0.1524" layer="91"/>
+<wire x1="38.1" y1="76.2" x2="38.1" y2="88.9" width="0.1524" layer="91"/>
 <pinref part="R1" gate="G$1" pin="2"/>
 <junction x="38.1" y="76.2"/>
-<pinref part="JP3" gate="A" pin="1"/>
+<wire x1="38.1" y1="88.9" x2="99.06" y2="88.9" width="0.1524" layer="91"/>
+<wire x1="99.06" y1="88.9" x2="99.06" y2="63.5" width="0.1524" layer="91"/>
+<pinref part="JP3" gate="A" pin="10"/>
+<wire x1="99.06" y1="63.5" x2="116.84" y2="63.5" width="0.1524" layer="91"/>
 </segment>
 </net>

Commit message: Agregue las fotos nuevas de las plaquetas y agregue la lista de componentes al word
Parts:
- R1: value (none) -> 10K
Changed lines of the file:
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@@
 <part name="SUPPLY8" library="supply2" library_urn="urn:adsk.eagle:library:372" deviceset="GND" device=""/>
 <part name="SUPPLY9" library="supply2" library_urn="urn:adsk.eagle:library:372" deviceset="GND" device=""/>
-<part name="R1" library="rcl" deviceset="R-EU_" device="0207/10" package3d_urn="urn:adsk.eagle:package:23491/2"/>
+<part name="R1" library="rcl" deviceset="R-EU_" device="0207/10" package3d_urn="urn:adsk.eagle:package:23491/2" value="10K"/>
 <part name="FRAME1" library="frames" library_urn="urn:adsk.eagle:library:229" deviceset="DINA4_L" device=""/>
 <part name="JP3" library="pinhead" deviceset="PINHD-1X16" device="" package3d_urn="urn:adsk.eagle:package:22432/2"/>
